Commit message: camera implemented inside gazebo

File: src/moveit/config/ur.gazebo_control.xacro (robot description, xacro)
@@ -1,4 +1,72 @@
 <?xml version="1.0"?>
 <robot xmlns:xacro="http://www.ros.org/wiki/xacro">
+  <!-- Test Object -->
+  <link name="test_obj_link">
+    <visual>
+      <origin xyz="0 0 1" rpy="0 0 0"/> <geometry>
+        <cylinder radius="1.0" length="2.0"/>
+      </geometry>
+      <material name="bright_red">
+        <color rgba="1 0 0 1"/>
+      </material>
+    </visual>
+    <collision>
+      <origin xyz="0 0 1" rpy="0 0 0"/>
+      <geometry>
+        <cylinder radius="1.0" length="2.0"/>
+      </geometry>
+    </collision>
+    <inertial>
+      <mass value="1.0"/>
+      <inertia ixx="0.41" ixy="0" ixz="0" iyy="0.41" iyz="0" izz="0.5"/>
+    </inertial>
+  </link>
+  <joint name="test_obj_joint" type="fixed">
+    <parent link="world"/>
+    <child link="test_obj_link"/>
+    <origin xyz="0 5 0" rpy="0 0 0"/>
+  </joint>
+  <!-- Camera -->
+  <link name="camera_link">
+    <visual>
+      <origin xyz="0 0 0" rpy="0 1.5707 0"/>
+      <geometry><cylinder radius="0.025" length="0.05"/></geometry>
+    </visual>
+    <collision>
+      <origin xyz="0 0 0" rpy="0 1.5707 0"/>
+      <geometry><cylinder radius="0.025" length="0.05"/></geometry>
+    </collision>
+  </link>
+  <joint name="camera_joint" type="fixed">
+    <parent link="wrist_2_link"/>
+    <child link="camera_link"/>
+    <origin xyz="0 0 0.075" rpy="0 0 1.5707"/>
+  </joint>
+  <gazebo reference="camera_link">
+    <sensor type="camera" name="sensor_camera">
+      <camera name="camera">
+        <image>
+          <width>320</width>
+          <height>240</height>
+        </image>
+        <horizontal_fov>1.05</horizontal_fov>
+        <clip>
+          <near>0.1</near>
+          <far>100.0</far>
+        </clip>
+      </camera>
+      <!-- <topic>camera</topic>  -->
+      <always_on>1</always_on>
+      <update_rate>30</update_rate>
+      <visualize>true</visualize>
+    </sensor>
+  </gazebo>
+  <gazebo>
+    <plugin filename="gz-sim-sensors-system"
+            name="gz::sim::systems::Sensors">
+      <render_engine>ogre2</render_engine>
+    </plugin>
+  </gazebo>
+  <!-- ROS2 Control -->
   <gazebo>
     <plugin filename="libgz_ros2_control-system.so" name="gz_ros2_control::GazeboSimROS2ControlPlugin">

Commit message: New world environment. Basic version with one tree

File: src/moveit/config/ur.gazebo_control.xacro (robot description, xacro)
@@ -1,30 +1,4 @@
 <?xml version="1.0"?>
 <robot xmlns:xacro="http://www.ros.org/wiki/xacro">
-  <!-- Test Object -->
-  <link name="test_obj_link">
-    <visual>
-      <origin xyz="0 0 1" rpy="0 0 0"/> <geometry>
-        <cylinder radius="1.0" length="2.0"/>
-      </geometry>
-      <material name="bright_red">
-        <color rgba="1 0 0 1"/>
-      </material>
-    </visual>
-    <collision>
-      <origin xyz="0 0 1" rpy="0 0 0"/>
-      <geometry>
-        <cylinder radius="1.0" length="2.0"/>
-      </geometry>
-    </collision>
-    <inertial>
-      <mass value="1.0"/>
-      <inertia ixx="0.41" ixy="0" ixz="0" iyy="0.41" iyz="0" izz="0.5"/>
-    </inertial>
-  </link>
-  <joint name="test_obj_joint" type="fixed">
-    <parent link="world"/>
-    <child link="test_obj_link"/>
-    <origin xyz="0 5 0" rpy="0 0 0"/>
-  </joint>
   <!-- Camera -->
   <link name="camera_link">
