Commit message: Arm and Scout are physically merged. However we still cannot operate them. They just exist as models inside Gazebo

File: src/manipulator/urdf/ur.urdf.xacro (robot description, xacro)
@@ -18,13 +18,19 @@
    <xacro:arg name="safety_pos_margin" default="0.15"/>
    <xacro:arg name="safety_k_position" default="20"/>
+   <!-- Origin Position -->
+   <xacro:arg name="origin_xyz" default="0 0 0"/>
    <!--When using gazebo simulations absolute paths are necessary.-->
    <xacro:arg name="force_abs_paths" default="false" />
-   <!-- create link fixed to the "world" -->
-   <link name="world" />
+   <xacro:arg name="arm_base_parent_link" default="world"/>
+   <xacro:property name="arm_base_parent_link" value="$(arg arm_base_parent_link)"/>
+   <!-- "world" link only for standalone use -->
+   <xacro:if value="${arm_base_parent_link == 'world'}">
+     <link name="world" />
+   </xacro:if>
    <!-- arm -->
    <xacro:ur_robot
      name="$(arg name)"
      tf_prefix="$(arg tf_prefix)"
-     parent="world"
+     parent="$(arg arm_base_parent_link)"
      joint_limits_parameters_file="$(arg joint_limit_params)"
      kinematics_parameters_file="$(arg kinematics_params)"
@@ -36,5 +42,5 @@
      force_abs_paths="$(arg force_abs_paths)"
      >
-     <origin xyz="0 0 0" rpy="0 0 0" />          <!-- position robot in the world -->
+     <origin xyz="$(arg origin_xyz)" rpy="0 0 0" />          <!-- position robot in the world -->
    </xacro:ur_robot>
 </robot>

File: src/moveit/config/ur.gazebo_control.xacro (robot description, xacro)
@@ -1,6 +1,7 @@
 <?xml version="1.0"?>
 <robot xmlns:xacro="http://www.ros.org/wiki/xacro">
+  <xacro:property name="tf_prefix" value="$(arg tf_prefix)"/>
   <!-- Camera -->
-  <link name="camera_link">
+  <link name="$(arg tf_prefix)camera_link">
     <visual>
       <origin xyz="0 0 0" rpy="0 1.5707 0"/>
@@ -12,13 +13,13 @@
     </collision>
   </link>
-  <joint name="camera_joint" type="fixed">
-    <parent link="wrist_2_link"/>
-    <child link="camera_link"/>
+  <joint name="$(arg tf_prefix)camera_joint" type="fixed">
+    <parent link="$(arg tf_prefix)wrist_2_link"/>
+    <child link="$(arg tf_prefix)camera_link"/>
     <origin xyz="0 0 0.075" rpy="0 0 1.5707"/>
   </joint>
-  <gazebo reference="camera_link">
-    <sensor type="rgbd_camera" name="sensor_camera">
-      <gz_frame_id>camera_link</gz_frame_id>
-      <camera name="camera">
+  <gazebo reference="$(arg tf_prefix)camera_link">
+    <sensor type="rgbd_camera" name="$(arg tf_prefix)sensor_camera">
+      <gz_frame_id>${tf_prefix}camera_link</gz_frame_id>
+      <camera name="$(arg tf_prefix)camera">
         <horizontal_fov>1.05</horizontal_fov>
         <image>
@@ -58,5 +59,5 @@
         <plugin>gz_ros2_control/GazeboSimSystem</plugin>
       </hardware>
-      <joint name="shoulder_pan_joint">
+      <joint name="$(arg tf_prefix)shoulder_pan_joint">
         <command_interface name="position"/>
         <state_interface name="position">
@@ -64,5 +65,5 @@
         </state_interface>
       </joint>
-      <joint name="shoulder_lift_joint">
+      <joint name="$(arg tf_prefix)shoulder_lift_joint">
         <command_interface name="position"/>
         <state_interface name="position">
@@ -70,5 +71,5 @@
         </state_interface>
       </joint>
-      <joint name="elbow_joint">
+      <joint name="$(arg tf_prefix)elbow_joint">
         <command_interface name="position"/>
         <state_interface name="position">
@@ -76,5 +77,5 @@
         </state_interface>
       </joint>
-      <joint name="wrist_1_joint">
+      <joint name="$(arg tf_prefix)wrist_1_joint">
         <command_interface name="position"/>
         <state_interface name="position">
@@ -82,5 +83,5 @@
         </state_interface>
       </joint>
-      <joint name="wrist_2_joint">
+      <joint name="$(arg tf_prefix)wrist_2_joint">
         <command_interface name="position"/>
         <state_interface name="position">
@@ -88,5 +89,5 @@
         </state_interface>
       </joint>
-      <joint name="wrist_3_joint">
+      <joint name="$(arg tf_prefix)wrist_3_joint">
         <command_interface name="position"/>
         <state_interface name="position">

File: src/robot_description_cutter/urdf/robot_cutter.urdf.xacro (robot description, xacro)
@@ -24,3 +24,9 @@
         initial_positions="${xacro.load_yaml(initial_positions_file)}"
     />
+    <gazebo>
+        <plugin filename="gz_ros2_control-system"
+                name="gz_ros2_control::GazeboSimROS2ControlPlugin">
+            <parameters>$(find robot_description_cutter)/config/controllers.yaml</parameters>
+        </plugin>
+    </gazebo>
 </robot>
