Commit message: Added the diff_drive_plugin so the Scout URDF works inside Gazebo (new topic /cmd_vel created to control both linear and angular velocities). Had to fix the wheels axis since we are rotating the mesh when spawning the left side wheels (for symmetry purposes)

File: src/scout_ros2/scout_description/urdf/scout_v2.xacro (robot description, xacro)
@@ -61,8 +61,8 @@
         <origin xyz="${wheelbase/2} ${-track/2} ${wheel_vertical_offset}" rpy="3.14 0 0" />
     </xacro:scout_wheel_type1>
-    <xacro:scout_wheel_type2 wheel_prefix="front_left">
+    <xacro:scout_wheel_type2 wheel_prefix="front_left" axis_xyz="0 1 0">
         <origin xyz="${wheelbase/2} ${track/2} ${wheel_vertical_offset}" rpy="0 0 0" />
     </xacro:scout_wheel_type2>
-    <xacro:scout_wheel_type1 wheel_prefix="rear_left">
+    <xacro:scout_wheel_type1 wheel_prefix="rear_left" axis_xyz="0 1 0">
         <origin xyz="${-wheelbase/2} ${track/2} ${wheel_vertical_offset}" rpy="0 0 0" />
     </xacro:scout_wheel_type1>
@@ -70,3 +70,33 @@
         <origin xyz="${-wheelbase/2} ${-track/2} ${wheel_vertical_offset}" rpy="3.14 0 0" />
     </xacro:scout_wheel_type2>
+    <!-- Gazebo: differential drive controller -->
+    <gazebo>
+        <plugin filename="gz-sim-diff-drive-system"
+                name="gz::sim::systems::DiffDrive">
+            <left_joint>front_left_wheel</left_joint>
+            <left_joint>rear_left_wheel</left_joint>
+            <right_joint>front_right_wheel</right_joint>
+            <right_joint>rear_right_wheel</right_joint>
+            <wheel_separation>${track}</wheel_separation>
+            <wheel_radius>${wheel_radius}</wheel_radius>
+            <odom_publish_frequency>50</odom_publish_frequency>
+            <topic>/cmd_vel</topic>
+            <odom_topic>/odom</odom_topic>
+            <tf_topic>/tf</tf_topic>
+            <frame_id>odom</frame_id>
+            <child_frame_id>base_link</child_frame_id>
+            <max_linear_acceleration>1</max_linear_acceleration>
+        </plugin>
+    </gazebo>
+    <!-- Gazebo: wheel joint state publisher -->
+    <gazebo>
+        <plugin filename="gz-sim-joint-state-publisher-system"
+                name="gz::sim::systems::JointStatePublisher">
+            <topic>/joint_states</topic>
+            <joint_name>front_left_wheel</joint_name>
+            <joint_name>front_right_wheel</joint_name>
+            <joint_name>rear_left_wheel</joint_name>
+            <joint_name>rear_right_wheel</joint_name>
+        </plugin>
+    </gazebo>
 </robot>

File: src/scout_ros2/scout_description/urdf/scout_wheel_type1.xacro (robot description, xacro)
@@ -24,5 +24,5 @@
 -->
 <robot xmlns:xacro="http://ros.org/wiki/xacro" name="scout_wheel">
-    <xacro:macro name="scout_wheel_type1" params="wheel_prefix *joint_pose">
+    <xacro:macro name="scout_wheel_type1" params="wheel_prefix axis_xyz:='0 -1 0' *joint_pose">
         <link name="${wheel_prefix}_wheel_link">
             <inertial>
@@ -44,9 +44,15 @@
             </collision>
         </link>
-        <joint name="${wheel_prefix}_wheel" type="fixed">
+        <!-- <joint name="${wheel_prefix}_wheel" type="fixed">
             <parent link="base_link"/>
             <child link="${wheel_prefix}_wheel_link"/>
             <xacro:insert_block name="joint_pose"/>
             <axis xyz="0 -1 0" rpy="0 0 0" />
+        </joint> -->
+        <joint name="${wheel_prefix}_wheel" type="continuous">
+            <parent link="base_link"/>
+            <child link="${wheel_prefix}_wheel_link"/>
+            <xacro:insert_block name="joint_pose"/>
+            <axis xyz="${axis_xyz}" rpy="0 0 0" />
         </joint>
     </xacro:macro>

File: src/scout_ros2/scout_description/urdf/scout_wheel_type2.xacro (robot description, xacro)
@@ -24,5 +24,5 @@
 -->
 <robot xmlns:xacro="http://ros.org/wiki/xacro" name="scout_wheel">
-    <xacro:macro name="scout_wheel_type2" params="wheel_prefix *joint_pose">
+    <xacro:macro name="scout_wheel_type2" params="wheel_prefix axis_xyz:='0 -1 0' *joint_pose">
         <link name="${wheel_prefix}_wheel_link">
             <inertial>
@@ -44,9 +44,15 @@
             </collision>
         </link>
-        <joint name="${wheel_prefix}_wheel" type="fixed">
+        <!-- <joint name="${wheel_prefix}_wheel" type="fixed">
             <parent link="base_link"/>
             <child link="${wheel_prefix}_wheel_link"/>
             <xacro:insert_block name="joint_pose"/>
             <axis xyz="0 -1 0" rpy="0 0 0" />
+        </joint> -->
+        <joint name="${wheel_prefix}_wheel" type="continuous">
+            <parent link="base_link"/>
+            <child link="${wheel_prefix}_wheel_link"/>
+            <xacro:insert_block name="joint_pose"/>
+            <axis xyz="${axis_xyz}" rpy="0 0 0" />
         </joint>
     </xacro:macro>
